File: GuitarPico/GuitarPico.kicad_pcb (KiCad board)
At the start: 2 copper layers, 100 x 100 mm, 125 parts, among them J1 INPUT, J2 INPUT, J3 OUTPUT, J4 OUTPUT, J5 Barrel_Jack_Switch, J6 VGA, J8 INPUT, J9 INPUT, Q1 2N3904, Q2 2N3904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

Commit message: Added simulations
Parts:
- C12: value 220 pF -> 2200 pF
- C13: value 220 pF -> 470 pF
- C8: value 330 nF -> 2200 pF
- C9: value 100 pF -> 47 pF
- R10, R9: value 1k -> 10k
- R11: value 10k -> 100k
- R13: value 10k -> 220k
Changed lines of the file:
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@@
       (effects (font (size 1 1) (thickness 0.15)))
     )
-    (fp_text value "1k" (at 3.81 2.37) (layer "F.Fab")
+    (fp_text value "10k" (at 3.81 2.37) (layer "F.Fab")
       (effects (font (size 1 1) (thickness 0.15)))
     )
@@
       (effects (font (size 1 1) (thickness 0.15)))
     )
-    (fp_text value "1k" (at 3.81 2.37) (layer "F.Fab")
+    (fp_text value "10k" (at 3.81 2.37) (layer "F.Fab")
       (effects (font (size 1 1) (thickness 0.15)))
     )
@@
       (effects (font (size 1 1) (thickness 0.15)))
     )
-    (fp_text value "220 pF" (at 2.5 2.5 90) (layer "F.Fab")
+    (fp_text value "2200 pF" (at 2.5 2.5 90) (layer "F.Fab")
       (effects (font (size 1 1) (thickness 0.15)))
     )
@@
       (effects (font (size 1 1) (thickness 0.15)))
     )
-    (fp_text value "330 nF" (at 2.5 2.5 90) (layer "F.Fab")
+    (fp_text value "2200 pF" (at 2.5 2.5 90) (layer "F.Fab")
       (effects (font (size 1 1) (thickness 0.15)))
     )
@@
       (effects (font (size 1 1) (thickness 0.15)))
     )
-    (fp_text value "10k" (at 3.81 2.37) (layer "F.Fab")
+    (fp_text value "100k" (at 3.81 2.37) (layer "F.Fab")
       (effects (font (size 1 1) (thickness 0.15)))
     )
@@
       (effects (font (size 1 1) (thickness 0.15)))
     )
-    (fp_text value "220 pF" (at 2.5 2.5 90) (layer "F.Fab")
+    (fp_text value "470 pF" (at 2.5 2.5 90) (layer "F.Fab")
       (effects (font (size 1 1) (thickness 0.15)))
     )
@@
       (effects (font (size 1 1) (thickness 0.15)))
     )
-    (fp_text value "10k" (at 3.81 2.37 90) (layer "F.Fab")
+    (fp_text value "220k" (at 3.81 2.37 90) (layer "F.Fab")
       (effects (font (size 1 1) (thickness 0.15)))
     )
@@
       (effects (font (size 1 1) (thickness 0.15)))
     )
-    (fp_text value "100 pF" (at 2.5 2.5) (layer "F.Fab")
+    (fp_text value "47 pF" (at 2.5 2.5) (layer "F.Fab")
       (effects (font (size 1 1) (thickness 0.15)))
     )
