File: StompBox/StompBox.kicad_pcb (KiCad board)
At the start: 2 copper layers, 207 x 52 mm, 43 parts, among them J1 AudioJack2_Dual_Ground_Switch, J2 Barrel_Jack_Switch, J3 Conn_01x03, J4 AudioJack2_Dual_Ground_Switch, J5 BATT, SW1 ThreeWayStompBox, SW2 ThreeWayStompBox, SW3 ThreeWayStompBox, SW4 ThreeWayStompBox

Commit message: Stompbox JLCPCB
Parts:
- added H10: MountingHole, MountingHole:MountingHole_3.2mm_M3, F.Cu at (165.3, 85.6)
- added H11: MountingHole, MountingHole:MountingHole_3.2mm_M3, F.Cu at (216.3, 85.1)
- added H12: MountingHole, MountingHole:MountingHole_3.2mm_M3, F.Cu at (64.3, 85.6)
- added H9: MountingHole, MountingHole:MountingHole_3.2mm_M3, F.Cu at (114.3, 85.6)
- added J6: AudioJack2_Dual_Ground_Switch, StompBox:PJ-3240-35mm-stereo, F.Cu at (46.3, 78.0)
- added R14: 10k, Resistor_THT:R_Axial_DIN0207_L6.3mm_D2.5mm_P7.62mm_Horizontal, F.Cu at (49.9, 93.7)
- moved R9 40.7 mm to (195.9, 96.6), turned to -90 degrees
- moved R8 31.7 mm to (231.9, 79.9), turned to 180 degrees
- moved R7 30.8 mm to (236.8, 107.6)
- moved C3 3.02 mm to (238.3, 110.9)
- moved J5 2.46 mm to (203.3, 65.8)
- moved R2 2.42 mm to (216.8, 69.6)
- moved R3 2.34 mm to (216.8, 73.0)
- moved RV1 2.15 mm to (215.8, 65.0)
- moved R13 1.62 mm to (49.9, 96.6)
- moved R1 0.90 mm to (231.4, 83.6)
Connections:
- C1 pad 1: OUTVOLT -> INVOLT
- C3 pad 1: Net-(SW4-Pad1P) -> Net-(C3-Pad1)
- J1 pad T1: OUTVOLT -> INVOLT
- J3 pad 2: OUTVOLT -> INVOLT
- J4 pad T1: Net-(SW4-Pad1P) -> Net-(C3-Pad1)
- JP1 pad 2: Net-(R7-Pad1) -> Net-(JP1-Pad2)
- JP2 pad 1: OUTVOLT -> INVOLT
- R7 pad 1: Net-(R7-Pad1) -> Net-(C3-Pad1)
- R8 pad 1: Net-(R7-Pad1) -> Net-(JP1-Pad2)
- R8 pad 2: Net-(SW4-Pad1P) -> Net-(C3-Pad1)
- SW1 pad 1P: Net-(SW4-Pad1P) -> Net-(C3-Pad1)
- SW2 pad 1P: Net-(SW4-Pad1P) -> Net-(C3-Pad1)
- SW3 pad 1P: Net-(SW4-Pad1P) -> Net-(C3-Pad1)
- SW4 pad 1P: Net-(SW4-Pad1P) -> Net-(C3-Pad1)
Routing:
- net Net-(C3-Pad1): track 0.00 -> 283.0 mm
- net Net-(SW4-Pad1P): track 229.3 -> 0.00 mm
- net INVOLT: track 45.4 -> 131.3 mm
- net Net-(R7-Pad1): track 58.3 -> 0.00 mm
- net OUTVOLT: track 51.9 -> 0.00 mm
- net +9V: track 276.9 -> 292.7 mm
- net Net-(R9-Pad2): track 13.6 -> 26.6 mm
- net Net-(R6-Pad2): track 42.1 -> 55.0 mm
- net Net-(J6-PadT1): track 0.00 -> 4.37 mm
- net Net-(JP1-Pad2): track 0.00 -> 4.35 mm
- net Net-(R4-Pad2): track 42.3 -> 46.2 mm
- net Net-(R5-Pad2): track 43.0 -> 46.0 mm
- net Net-(J1-PadS1): track 60.5 -> 58.5 mm
- net Net-(R3-Pad1): track 24.5 -> 26.5 mm
- net Net-(J4-PadS1): track 34.4 -> 33.4 mm
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Other:
- board text added: "VOLUME INPUT"
